Commit message: added some urdf files

File: src/models/micromouse_robot.urdf (robot description, URDF)
Before this commit: robot my_mm_robot, 3 links, 2 joints
Links:
- added link sensor_laser, mass 0.01; collision cylinder length=0.001 radius=0.005; visual cylinder length=0.02 radius=0.005
Joints:
- added joint joint_sensor_laser: type fixed, parent link_chassis, child sensor_laser, origin xyz=0    0    0.01 rpy=0  0  -1.57
