Commit message: added test3, which is basically swarm start

File: omni3ros_pkg/urdf/main3.urdf.xacro (robot description, xacro)
@@ -1,5 +1,4 @@
 <?xml version="1.0"?>
 <robot xmlns:xacro="http://www.ros.org/wiki/xacro" name="open_base">
-	<xacro:property name="namespace" value="$(arg namespace)" />
 	<xacro:include filename="$(find omni3ros_pkg)/urdf/rim.urdf.xacro"/>
 	<link name="origin_link"/>
@@ -63,5 +62,5 @@
 	<gazebo>
 		<plugin name="gazebo_ros_control" filename="libgazebo_ros_control.so">
-		<robotNamespace>$(arg namespace)</robotNamespace>
+		<robotNamespace>/open_base</robotNamespace>
 		</plugin>
 	</gazebo>
@@ -115,5 +114,5 @@
       </ray>
       <plugin name="gazebo_ros_head_hokuyo_controller" filename="libgazebo_ros_laser.so">
-        <topicName>/$(arg namespace)/laser/scan</topicName>
+        <topicName>/laser/scan</topicName>
         <frameName>base_link</frameName>
       </plugin>
