Commit message: added new mesh file with our bot and laser sensor

File: omni3ros_pkg/urdf/main2.urdf.xacro (robot description, xacro)
@@ -65,3 +65,58 @@
 		</plugin>
 	</gazebo>
+  <!--
+    Adding a laser scan sensor to the robot
+  -->
+  <link name="sensor_laser">
+    <inertial>
+      <origin xyz="0 0 0" rpy="0 0 0" />
+      <mass value="0.01" />
+      <inertia ixx="0.02" ixy="0" ixz="0" iyy="0.02" iyz="0" izz="0.02"/>
+    </inertial>
+    <visual>
+      <origin xyz="0.00 0 0.0" rpy="0 0 0" />
+      <geometry>
+        <cylinder radius="0.005" length="0.02"/>
+      </geometry>
+      <material name="Red" />
+    </visual>
+    <collision>
+      <origin xyz="0 0 0" rpy="0 0 0"/>
+      <geometry>
+        <cylinder radius="0.005" length="0.001"/>
+      </geometry>
+    </collision>
+  </link>
+  <joint name="joint_sensor_laser" type="fixed">
+    <origin rpy="0  0  1.570796" xyz="0    0    0.09"/>
+    <parent link="base_link"/>
+    <child link="sensor_laser"/>
+  </joint>
+  <gazebo reference="sensor_laser">
+    <sensor type="ray" name="head_hokuyo_sensor">
+      <pose>0 0 0 0 0 0</pose>
+      <visualize>true</visualize>
+      <update_rate>20</update_rate>
+      <ray>
+        <scan>
+          <horizontal>
+            <samples>360</samples>
+            <resolution>1</resolution>
+            <min_angle>-1.570796</min_angle>
+            <max_angle>1.570796</max_angle>
+          </horizontal>
+        </scan>
+        <range>
+          <min>0.172</min>
+          <max>10.0</max>
+          <resolution>0.01</resolution>
+        </range>
+      </ray>
+      <plugin name="gazebo_ros_head_hokuyo_controller" filename="libgazebo_ros_laser.so">
+	<robotNamespace>open_base</robotNamespace>
+        <topicName>/open_base/laser/scan</topicName>
+        <frameName>base_link</frameName>
+      </plugin>
+    </sensor>
+  </gazebo>
 </robot>

Commit message: Fixed sensor frame wrt base which caused wrong maps

File: omni3ros_pkg/urdf/main2.urdf.xacro (robot description, xacro)
@@ -89,5 +89,5 @@
   </link>
   <joint name="joint_sensor_laser" type="fixed">
-    <origin rpy="0  0  1.570796" xyz="0    0    0.09"/>
+    <origin rpy="0  0  0" xyz="0    0    0.09"/>
     <parent link="base_link"/>
     <child link="sensor_laser"/>
@@ -103,6 +103,6 @@
             <samples>360</samples>
             <resolution>1</resolution>
-            <min_angle>-1.570796</min_angle>
-            <max_angle>1.570796</max_angle>
+            <min_angle>0</min_angle>
+            <max_angle>3.14159</max_angle>
           </horizontal>
         </scan>

Commit message: yeah

File: omni3ros_pkg/urdf/main2.urdf.xacro (robot description, xacro)
@@ -6,12 +6,6 @@
 	<link name="base_link">
 	<inertial>
-		<mass value="0.07862944645"/>
-		<inertia
-			ixx="0.00002035985530754"
-			ixy="0"
-			ixz="0"
-			iyy="0.00002035985530754"
-			iyz="0"
-			izz="0.00003945961663220"/>
+		<mass value="2.4"/>
+		<inertia ixx="0.02534" ixy="0" ixz="0" iyy="0.02534" iyz="0" izz="0.03468"/>
 		</inertial>
 	<visual>

Commit message: Things to change : \nNeed to coorect the des ang prob.. and need to correct why is it going back..

File: omni3ros_pkg/urdf/main2.urdf.xacro (robot description, xacro)
@@ -6,6 +6,12 @@
 	<link name="base_link">
 	<inertial>
-		<mass value="2.4"/>
-		<inertia ixx="0.02534" ixy="0" ixz="0" iyy="0.02534" iyz="0" izz="0.03468"/>
+		<mass value="0.07862944645"/>
+		<inertia
+			ixx="0.00002035985530754"
+			ixy="0"
+			ixz="0"
+			iyy="0.00002035985530754"
+			iyz="0"
+			izz="0.00003945961663220"/>
 		</inertial>
 	<visual>
